Commit message: fix gps bug!!!!

File: models/lequad/urdf/component_snippets.xacro (robot description, xacro)
@@ -108,16 +108,16 @@
   <xacro:macro name="controller_plugin_macro" params="namespace imu_sub_topic">
     <gazebo>
-      <plugin name="controller_interface" filename="libgazebo_controller_interface.so">
-        <robotNamespace>${namespace}</robotNamespace>
-        <commandAttitudeThrustSubTopic>/command/attitude</commandAttitudeThrustSubTopic>
-        <commandRateThrustSubTopic>/command/rate</commandRateThrustSubTopic>
-        <commandMotorSpeedSubTopic>/command/motor_speed</commandMotorSpeedSubTopic>
-        <imuSubTopic>/${imu_sub_topic}</imuSubTopic>
-        <motorSpeedCommandPubTopic>/gazebo/command/motor_speed</motorSpeedCommandPubTopic>
-      </plugin>
+        <plugin name="controller_interface" filename="libgazebo_controller_interface.so">
+          <robotNamespace>${namespace}</robotNamespace>
+          <commandAttitudeThrustSubTopic>/command/attitude</commandAttitudeThrustSubTopic>
+          <commandRateThrustSubTopic>/command/rate</commandRateThrustSubTopic>
+          <commandMotorSpeedSubTopic>/command/motor_speed</commandMotorSpeedSubTopic>
+          <imuSubTopic>/${imu_sub_topic}</imuSubTopic>
+          <motorSpeedCommandPubTopic>/gazebo/command/motor_speed</motorSpeedCommandPubTopic>
+        </plugin>
     </gazebo>
   </xacro:macro>
   <!-- Macro to add the gps_plugin. -->
-  <xacro:macro name="gps_plugin_macro" params="namespace gps_noise">
+  <!-- <xacro:macro name="gps_plugin_macro" params="namespace gps_noise">
     <gazebo>
       <plugin name="gps_plugin" filename="libgazebo_gps_plugin.so">
@@ -126,4 +126,64 @@
       </plugin>
     </gazebo>
+  </xacro:macro> -->
+  <xacro:macro name="gps_plugin_macro" params="namespace gps_noise">
+    <gazebo>
+      <model name='gps0'>
+        <link name='link'>
+          <pose>0 0 0 0 0 0</pose>
+          <inertial>
+            <pose>0 0 0 0 0 0</pose>
+            <mass>0.01</mass>
+            <inertia>
+              <ixx>2.1733e-06</ixx>
+              <ixy>0</ixy>
+              <ixz>0</ixz>
+              <iyy>2.1733e-06</iyy>
+              <iyz>0</iyz>
+              <izz>1.8e-07</izz>
+            </inertia>
+          </inertial>
+          <visual name='visual'>
+            <geometry>
+              <cylinder>
+                <radius>0.01</radius>
+                <length>0.002</length>
+              </cylinder>
+            </geometry>
+            <material>
+              <script>
+                <name>Gazebo/Black</name>
+                <uri>__default__</uri>
+              </script>
+            </material>
+          </visual>
+          <sensor name="gps" type="gps">
+            <pose>0 0 0 0 0 0</pose>
+            <plugin name="gps_plugin" filename="libgazebo_gps_plugin.so">
+              <robotNamespace>${namespace}</robotNamespace>
+              <gpsNoise>${gps_noise}</gpsNoise>
+              <gpsXYRandomWalk>2.0</gpsXYRandomWalk>
+              <gpsZRandomWalk>4.0</gpsZRandomWalk>
+              <gpsXYNoiseDensity>0.0002</gpsXYNoiseDensity>
+              <gpsZNoiseDensity>0.0004</gpsZNoiseDensity>
+              <gpsVXYNoiseDensity>0.2</gpsVXYNoiseDensity>
+              <gpsVZNoiseDensity>0.4</gpsVZNoiseDensity>
+            </plugin>
+          </sensor>
+        </link>
+      </model>
+    </gazebo>
+    <!-- <gazebo reference="gps0::link">
+        <material>
+              <script>
+                <name>Gazebo/Black</name>
+                <uri>__default__</uri>
+              </script>
+      </material>
+    </gazebo>
+    <joint name='gps0_joint' type='fixed'>
+        <parent link="base_link"/>
+        <child link="gps0::link"/>
+    </joint> -->
   </xacro:macro>
   <!-- Macro to add the magnetometer_plugin. -->
